Commit message: nero_both_arms dual arm control with gripper

File: examples/nero_both_arms/antt_t1.urdf (robot description, URDF)
Before this commit: robot antt_t1, 20 links, 19 joints
Links:
- added link left_gripper_base, mass 0.45; collision mesh filename=meshes/gripper_base.stl; visual mesh filename=meshes/dae/gripper_base.dae
- added link left_gripper_flange, mass 0.04771096; collision mesh filename=meshes/gripper_flange.stl; visual mesh filename=meshes/dae/gripper_flange.dae
- added link left_gripper_link1, mass 0.025; collision mesh filename=meshes/gripper_link1.stl; visual mesh filename=meshes/dae/gripper_link1.dae
- added link left_gripper_link2, mass 0.025; collision mesh filename=meshes/gripper_link2.stl; visual mesh filename=meshes/dae/gripper_link2.dae
- added link right_gripper_base, mass 0.45; collision mesh filename=meshes/gripper_base.stl; visual mesh filename=meshes/dae/gripper_base.dae
- added link right_gripper_flange, mass 0.04771096; collision mesh filename=meshes/gripper_flange.stl; visual mesh filename=meshes/dae/gripper_flange.dae
- added link right_gripper_link1, mass 0.025; collision mesh filename=meshes/gripper_link1.stl; visual mesh filename=meshes/dae/gripper_link1.dae
- added link right_gripper_link2, mass 0.025; collision mesh filename=meshes/gripper_link2.stl; visual mesh filename=meshes/dae/gripper_link2.dae
- link left_link8: mass None -> 0.05; geometry collision mesh filename=package://nero_description/meshes/stand_v1.dae; visual mesh filename=package://nero_description/meshes/stand_v1.dae
- link right_link8: mass None -> 0.05; geometry collision mesh filename=package://nero_description/meshes/stand_v1.dae; visual mesh filename=package://nero_description/meshes/stand_v1.dae
Joints:
- added joint left_gripper_base_joint: type fixed, parent left_gripper_flange, child left_gripper_base, origin xyz=0 0 0.0055 rpy=0 0 0
- added joint left_gripper_flange_joint: type fixed, parent left_link7, child left_gripper_flange, origin xyz=0.032 0 -0.0235 rpy=-1.5708 0 -1.5708
- added joint left_gripper_joint1: type prismatic, parent left_gripper_base, child left_gripper_link1, origin xyz=0 0 0.1358 rpy=1.5707963 0 3.1415926, axis 0 0 1, limit lower=0 upper=0.05 effort=10 velocity=3
- added joint left_gripper_joint2: type prismatic, parent left_gripper_base, child left_gripper_link2, origin xyz=0 0 0.1358 rpy=1.5707963 0 0, axis 0 0 -1, limit lower=-0.05 upper=0 effort=10 velocity=3
- added joint right_gripper_base_joint: type fixed, parent right_gripper_flange, child right_gripper_base, origin xyz=0 0 0.0055 rpy=0 0 0
- added joint right_gripper_flange_joint: type fixed, parent right_link7, child right_gripper_flange, origin xyz=0.032 0 -0.0235 rpy=-1.5708 0 -1.5708
- added joint right_gripper_joint1: type prismatic, parent right_gripper_base, child right_gripper_link1, origin xyz=0 0 0.1358 rpy=1.5707963 0 3.1415926, axis 0 0 1, limit lower=0 upper=0.05 effort=10 velocity=3
- added joint right_gripper_joint2: type prismatic, parent right_gripper_base, child right_gripper_link2, origin xyz=0 0 0.1358 rpy=1.5707963 0 0, axis 0 0 -1, limit lower=-0.05 upper=0 effort=10 velocity=3
- joint left_joint8: origin xyz=0.00000000 0.00000000 -0.02350000 rpy=0 0 0 -> xyz=0.033 0.00000000 -0.02350000 rpy=0 0 0
- joint right_joint8: origin xyz=0.00000000 0.00000000 -0.02350000 rpy=0 0 0 -> xyz=0.033 0.00000000 -0.02350000 rpy=0 0 0
